File: pcb/powersupply.kicad_sch (KiCad schematic)
At the start: 28 parts, among them J1 Conn_01x02_Pin, U1 LD39200PU33R, U2 MIC26903YJL-TR, U3 INA219AIDCNR

Commit message: first commit
Parts:
- R2: value 560 -> 240
Other:
- note added: "Based on typical application in datasheet"
- note added: "Fixed Version"
- note added: "I2C Address: 0x40"
- note added: "Vout = 0.8 * (1 + R6/R7)"
Changed lines of the file:
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@@
 		)
 	)
+	(text "Based on typical application in datasheet"
+		(exclude_from_sim no)
+		(at 114.3 131.064 0)
+		(effects
+			(font
+				(size 1.27 1.27)
+			)
+		)
+	)
+	(text "I2C Address: 0x40"
+		(exclude_from_sim no)
+		(at 229.108 55.88 0)
+		(effects
+			(font
+				(size 1.27 1.27)
+			)
+		)
+	)
 	(text "Raw Input"
 		(exclude_from_sim no)
@@
 		)
 	)
+	(text "Fixed Version"
+		(exclude_from_sim no)
+		(at 88.646 184.15 0)
+		(effects
+			(font
+				(size 1.27 1.27)
+			)
+		)
+	)
 	(text "Power Supply System"
 		(exclude_from_sim no)
@@
 		)
 	)
+	(text "Vout = 0.8 * (1 + R6/R7)"
+		(exclude_from_sim no)
+		(at 214.884 131.064 0)
+		(effects
+			(font
+				(size 1.27 1.27)
+			)
+		)
+	)
 	(junction
 		(at 248.92 100.33)
@@
 			)
 		)
-		(property "Value" "560"
+		(property "Value" "240"
 			(at 138.43 180.3399 0)
 			(effects
